Commit message: updated

File: install/braccio_description/share/braccio_description/urdf/braccio.urdf.xacro (robot description, xacro)
@@ -140,4 +140,7 @@
       <material name="white"/>
     </visual>
+    <collision>
+      <geometry><sphere radius="0.005"/></geometry>
+    </collision>
     <inertial>
       <mass value="0.001"/>
@@ -220,4 +223,10 @@
   <!-- ==================== GAZEBO ==================== -->
   <gazebo>
+    <plugin filename="libgz-sim-sensors-system.so" name="gz::sim::systems::Sensors">
+      <render_engine>ogre2</render_engine>
+    </plugin>
+  </gazebo>
+  <!-- ROS2 Control -->
+  <gazebo>
     <plugin filename="gz_ros2_control-system" name="gz_ros2_control::GazeboSimROS2ControlPlugin">
       <robot_param>robot_description</robot_param>
@@ -226,8 +235,11 @@
     </plugin>
   </gazebo>
+  <!-- Camera sensor - FIXED: proper plugin opening tag -->
   <gazebo reference="camera_link">
     <sensor name="workspace_camera" type="camera">
       <always_on>true</always_on>
       <update_rate>30</update_rate>
+      <visualize>true</visualize>
+      <topic>camera</topic>
       <camera>
         <horizontal_fov>1.047</horizontal_fov>
@@ -235,14 +247,7 @@
         <clip><near>0.01</near><far>10.0</far></clip>
       </camera>
-      <plugin filename="gz-sim-camera-system" name="gz::sim::systems::Camera">
-        <ros>
-          <remapping>~/image_raw:=/camera/image_raw</remapping>
-          <remapping>~/camera_info:=/camera/camera_info</remapping>
-        </ros>
-        <camera_name>workspace_camera</camera_name>
-        <frame_name>camera_optical_link</frame_name>
-      </plugin>
     </sensor>
   </gazebo>
+  <!-- Gazebo materials -->
   <gazebo reference="base_link"><material>Gazebo/Black</material></gazebo>
   <gazebo reference="braccio_base_link"><material>Gazebo/Gray</material></gazebo>

Commit message: Real pixel-to-world detection, elbow limit fix, IK seed reuse, grasp height fix

File: install/braccio_description/share/braccio_description/urdf/braccio.urdf.xacro (robot description, xacro)
@@ -7,4 +7,7 @@
   <material name="white"><color rgba="0.8 0.8 0.8 1.0"/></material>
   <material name="black"><color rgba="0 0 0 0.50"/></material>
+  <material name="red"><color rgba="0.8 0.0 0.0 1.0"/></material>
+  <material name="blue"><color rgba="0.0 0.0 0.8 1.0"/></material>
+  <material name="green"><color rgba="0.0 0.8 0.0 1.0"/></material>
   <!-- ==================== MACROS ==================== -->
   <xacro:macro name="braccio_link" params="name mesh_name color origin_xyz origin_rpy mass ixx iyy izz ixy ixz iyz">
@@ -157,5 +160,5 @@
     <visual>
       <geometry><box size="0.03 0.03 0.02"/></geometry>
-      <material name="black"/>
+      <material name="red"/>
     </visual>
     <collision>
@@ -182,5 +185,5 @@
   <xacro:braccio_revolute_joint name="elbow_joint"
     parent="shoulder_link" child="elbow_link"
-    axis_xyz="1 0 0" limit_lower="1.0" limit_upper="4.6"
+    axis_xyz="1 0 0" limit_lower="1.0" limit_upper="5.0"
     origin_xyz="0 0 0.125" origin_rpy="-2.8 0 0"/>
   <xacro:braccio_revolute_joint name="wrist_pitch_joint"
@@ -212,5 +215,5 @@
   <!-- CHANGED: Camera now attached to base_link instead of world -->
   <joint name="camera_joint" type="fixed">
-    <origin rpy="0 1.5708 0" xyz="0.30 0 0.59"/>
+    <origin rpy="0 1.5708 3.1416" xyz="0.30 0 0.59"/>
     <parent link="base_link"/>
     <child link="camera_link"/>
@@ -232,5 +235,5 @@
       <robot_param>robot_description</robot_param>
       <robot_param_node>robot_state_publisher</robot_param_node>
-      <parameters>$(find braccio_description)/config/braccio_controllers.yaml</parameters>
+      <parameters>/home/ubuntu/my_workspace/install/braccio_description/share/braccio_description/config/braccio_controllers.yaml</parameters>
     </plugin>
   </gazebo>
@@ -240,5 +243,5 @@
       <always_on>true</always_on>
       <update_rate>30</update_rate>
-      <visualize>true</visualize>
+      <visualize>false</visualize>
       <topic>camera</topic>
       <camera>

File: src/braccio_description/urdf/braccio.urdf.xacro (robot description, xacro)
@@ -185,5 +185,5 @@
   <xacro:braccio_revolute_joint name="elbow_joint"
     parent="shoulder_link" child="elbow_link"
-    axis_xyz="1 0 0" limit_lower="1.0" limit_upper="4.6"
+    axis_xyz="1 0 0" limit_lower="1.0" limit_upper="5.0"
     origin_xyz="0 0 0.125" origin_rpy="-2.8 0 0"/>
   <xacro:braccio_revolute_joint name="wrist_pitch_joint"
