Commit message: updated

File: src/braccio_description/urdf/braccio.urdf.xacro (robot description, xacro)
@@ -7,4 +7,7 @@
   <material name="white"><color rgba="0.8 0.8 0.8 1.0"/></material>
   <material name="black"><color rgba="0 0 0 0.50"/></material>
+  <material name="red"><color rgba="0.8 0.0 0.0 1.0"/></material>
+  <material name="blue"><color rgba="0.0 0.0 0.8 1.0"/></material>
+  <material name="green"><color rgba="0.0 0.8 0.0 1.0"/></material>
   <!-- ==================== MACROS ==================== -->
   <xacro:macro name="braccio_link" params="name mesh_name color origin_xyz origin_rpy mass ixx iyy izz ixy ixz iyz">
@@ -157,5 +160,5 @@
     <visual>
       <geometry><box size="0.03 0.03 0.02"/></geometry>
-      <material name="black"/>
+      <material name="red"/>
     </visual>
     <collision>
@@ -212,5 +215,5 @@
   <!-- CHANGED: Camera now attached to base_link instead of world -->
   <joint name="camera_joint" type="fixed">
-    <origin rpy="0 1.5708 0" xyz="0.30 0 0.59"/>
+    <origin rpy="0 1.5708 3.1416" xyz="0.30 0 0.59"/>
     <parent link="base_link"/>
     <child link="camera_link"/>

Commit message: removed hardcoding , according to logs , whole pick and place sequence works

File: src/braccio_description/urdf/braccio.urdf.xacro (robot description, xacro)
@@ -53,5 +53,5 @@
   </xacro:macro>
   <!-- ==================== LINKS ==================== -->
-  <!-- REMOVED: <link name="world"/> -->
+  <link name="world"/>
   <!-- Base Link: flat cylinder r=0.053, h=0.01, m=0.5
        NOW THE ROOT LINK - No world link above it
@@ -173,5 +173,9 @@
   <link name="camera_optical_link"/>
   <!-- ==================== JOINTS ==================== -->
-  <!-- REMOVED: world_joint -->
+  <joint name="world_joint" type="fixed">
+   <parent link="world"/>
+    <child link="base_link"/>
+   <origin xyz="0 0 0" rpy="0 0 0"/>
+ </joint>
   <!-- base_link is now the root, no parent above it -->
   <xacro:braccio_revolute_joint name="base_joint"
@@ -215,5 +219,5 @@
   <!-- CHANGED: Camera now attached to base_link instead of world -->
   <joint name="camera_joint" type="fixed">
-    <origin rpy="0 1.5708 3.1416" xyz="0.30 0 0.59"/>
+    <origin rpy="0 1.5708 3.1416" xyz="0.05 -0.15 0.59"/>
     <parent link="base_link"/>
     <child link="camera_link"/>
